Commit message: use stl collision model

File: robotino_description/urdf/base_old.urdf.xacro (robot description, xacro)
@@ -102,5 +102,5 @@
       <origin xyz="0.01 0 0.12" rpy="0 0 0"/>
       <geometry>
-       <cylinder length="0.24" radius="0.23"/>
+       <mesh filename="package://robotino_description/meshes/RobotinoBody.stl"/>
       </geometry>
     </collision>

Commit message: update collision models

File: robotino_description/urdf/base_old.urdf.xacro (robot description, xacro)
@@ -100,5 +100,5 @@
     </visual>
     <collision>
-      <origin xyz="0.01 0 0.12" rpy="0 0 0"/>
+      <origin xyz="0.01 0 0" rpy="0 0 0"/>
       <geometry>
        <mesh filename="package://robotino_description/meshes/RobotinoBody.stl"/>

File: robotino_description/urdf/hokuyo.urdf.xacro (robot description, xacro)
@@ -22,7 +22,7 @@
       </visual>
       <collision>
-        <origin xyz="0 0 ${HOKUYO_LENGTH/2}" rpy="0 0 0" />
+        <origin xyz="0 0 0.005" rpy="0 0 0" />
         <geometry>
-          <cylinder radius="${HOKUYO_RADIUS}" length="${HOKUYO_LENGTH}" />
+          <cylinder radius="0.01" length="0.01" />
         </geometry>
       </collision>
