Commit message: removed softlimits

File: robotino_description/urdf/base.urdf.xacro (robot description, xacro)
@@ -37,6 +37,4 @@
     <axis xyz="1 0 0" />
     <limit upper="10" lower="-10" effort="0" velocity="0" />
-    <dynamics damping="1000.0" friction="1000.0"/>
-    <safety_controller k_velocity="10" k_position="15" soft_lower_limit="-2.0" soft_upper_limit="0.5" />
    </joint>
    <joints_transmission name="base_jointx" />
@@ -47,6 +45,4 @@
     <axis xyz="0 1 0" />
     <limit upper="10" lower="-10" effort="0" velocity="0" />
-    <dynamics damping="1000.0" friction="1000.0"/>
-    <safety_controller k_velocity="10" k_position="15" soft_lower_limit="-2.0" soft_upper_limit="0.5" />
    </joint>
    <joints_transmission name="base_jointy" />
@@ -57,6 +53,4 @@
     <axis xyz="0 0 1" />
     <limit upper="3.14" lower="-3.14" effort="0" velocity="0" />
-    <dynamics damping="1000.0" friction="1000.0"/>
-    <safety_controller k_velocity="10" k_position="15" soft_lower_limit="-2.0" soft_upper_limit="0.5" />
    </joint>
    <joints_transmission name="base_jointz" />

Commit message: fixed joint velocity limits

File: robotino_description/urdf/base.urdf.xacro (robot description, xacro)
@@ -35,5 +35,5 @@
     <origin xyz="0 0 0" rpy="0 0 0" />
     <axis xyz="1 0 0" />
-    <limit upper="20" lower="-20" effort="0" velocity="0" />
+    <limit upper="20" lower="-20" effort="0" velocity="0.3" />
     <dynamics damping="1000.0" friction="1000.0"/>
     <safety_controller k_velocity="10" k_position="15" soft_lower_limit="-10.0" soft_upper_limit="10.0" />
@@ -45,5 +45,5 @@
     <origin xyz="0 0 0" rpy="0 0 0" />
     <axis xyz="0 1 0" />
-    <limit upper="20" lower="-20" effort="0" velocity="0" />
+    <limit upper="20" lower="-20" effort="0" velocity="0.3" />
     <dynamics damping="1000.0" friction="1000.0"/>
     <safety_controller k_velocity="10" k_position="15" soft_lower_limit="-10.0" soft_upper_limit="10.0" />
@@ -55,5 +55,5 @@
     <origin xyz="0 0 0" rpy="0 0 0" />
     <axis xyz="0 0 1" />
-    <limit upper="3.14" lower="-3.14" effort="0" velocity="0" />
+    <limit upper="3.14" lower="-3.14" effort="0" velocity="0.7" />
     <dynamics damping="1000.0" friction="1000.0"/>
     <safety_controller k_velocity="10" k_position="15" soft_lower_limit="-3.14" soft_upper_limit="3.14" />
