Commit message: first arm description

File: robotino_description/urdf/arm.urdf.xacro (robot description, xacro)
@@ -1,15 +1,186 @@
 <?xml version="1.0"?>
-<robot xmlns:xacro="http://www.ros.org/wiki/xacro">
-  <xacro:macro name="default_inertial">
-    <inertial>
-      <mass value="0.01"/>
-      <origin xyz="0 0 0"/>
-      <inertia ixx="0.001" ixy="0.0" ixz="0.0" iyy="0.001" iyz="0.0" izz="0.001" />
-    </inertial>
+<robot xmlns:xacro="http://wiki.ros.org/xacro">
+  <xacro:macro name="arm">
+    <link name="base">
+      <xacro:default_inertial/>
+      <visual>
+        <geometry>
+          <box size="0.04096 0.0473 0.105" />
+        </geometry>
+        <material name="white">
+          <color rgba="1 1 1 1"/>
+        </material>
+        <origin rpy="0 0 0" xyz="0 0 0.0525"/>
+      </visual>
+    </link>
+    <joint name="fixed_base_motor1" type="fixed">
+      <parent link="base"/>
+      <child link="motor1"/>
+      <axis xyz="0 0 1" />
+      <origin xyz="0.0 -0.01591 0.140" rpy="0 0 0" />
+      <limit upper="1.7" lower="-1.7" effort="160" velocity="30" />
+    </joint>
+    <link name="motor1">
+      <xacro:default_inertial/>
+      <visual>
+        <geometry>
+          <mesh filename="package://robotino_description/meshes/arm/motor1.stl"/>
+        </geometry>
+        <material name="white">
+          <color rgba="1 1 1 1"/>
+        </material>
+        <origin rpy="0 0 0" xyz="0 0 0."/>
+      </visual>
+      <collision>
+        <origin rpy="0 0 0" xyz="0 0 0."/>
+        <geometry>
+          <mesh filename="package://robotino_description/meshes/arm/motor1_collision.stl"/>
+        </geometry>
+      </collision>
+    </link>
+    <joint name="joint1" type="revolute">
+      <parent link="motor1"/>
+      <child link="link1"/>
+      <origin xyz="0.0 0.0 0.0" rpy="0 0 0" />
+      <axis xyz="0 1 0" />
+      <limit upper="1.9" lower="-1.9" effort="190" velocity="30" />
+    </joint>
+    <link name="link1">
+      <xacro:default_inertial/>
+      <visual>
+        <geometry>
+          <mesh filename="package://robotino_description/meshes/arm/link1.stl"/>
+        </geometry>
+        <material name="white" />
+        <origin rpy="0 0 0" xyz="0 0 0"/>
+      </visual>
+      <collision>
+        <origin rpy="0 0 0" xyz="0 0 0"/>
+        <geometry>
+          <mesh filename="package://robotino_description/meshes/arm/link1_collision.stl"/>
+        </geometry>
+      </collision>
+    </link>
+    <gazebo reference="link1">
+        <material>Gazebo/White</material>
+    </gazebo>
+    <joint name="joint2" type="revolute">
+      <parent link="link1"/>
+      <child link="motor2"/>
+      <origin xyz="0.0 0.09 0.28" rpy="0 0 0" />
+      <axis xyz="0 1 0" />
+      <limit upper="1.9" lower="-1.9" effort="190" velocity="30" />
+    </joint>
+    <link name="motor2">
+      <xacro:default_inertial/>
+      <visual>
+        <geometry>
+          <box size="0 0 0" />
+        </geometry>
+        <material name="white" />
+        <origin rpy="0 0 0" xyz="0 0.0625 0."/>
+      </visual>
+    </link>
+    <joint name="fixed_motor2_link2" type="fixed">
+      <parent link="motor2"/>
+      <child link="link2"/>
+      <origin xyz="0.0 0.098 0.027" rpy="0 0 0" />
+    </joint>
+    <link name="link2">
+      <xacro:default_inertial/>
+      <visual>
+        <geometry>
+          <mesh filename="package://robotino_description/meshes/arm/link2.stl"/>
+        </geometry>
+        <material name="white" />
+        <origin rpy="0 0 0" xyz="0 0 0"/>
+      </visual>
+      <collision>
+        <origin rpy="0 0 0" xyz="0 0 0"/>
+        <geometry>
+          <mesh filename="package://robotino_description/meshes/arm/link2_collision.stl"/>
+        </geometry>
+      </collision>
+    </link>
+    <gazebo reference="link2">
+      <material>Gazebo/White</material>
+    </gazebo>
+    <joint name="joint3" type="revolute">
+      <parent link="link2"/>
+      <child link="link3"/>
+      <origin xyz="0.0 0.0 0.13" rpy="0 0 0" />
+      <axis xyz="0 0 1" />
+      <limit upper="1.7" lower="-1.7" effort="190" velocity="30" />
+    </joint>
+    <link name="link3">
+      <xacro:default_inertial/>
+      <visual>
+        <geometry>
+          <mesh filename="package://robotino_description/meshes/arm/link3.stl"/>
+        </geometry>
+        <material name="white" />
+        <origin rpy="0 0 0" xyz="0 0 0"/>
+      </visual>
+      <collision>
+        <origin rpy="0 0 0" xyz="0 0 0"/>
+        <geometry>
+          <mesh filename="package://robotino_description/meshes/arm/link3_collision.stl"/>
+        </geometry>
+      </collision>
+    </link>
+    <gazebo reference="link3">
+      <material>Gazebo/White</material>
+    </gazebo>
+    <joint name="joint4" type="revolute">
+      <parent link="link3"/>
+      <child link="link4"/>
+      <origin xyz="0.0 -0.053 0.065" rpy="0 0 0" />
+      <axis xyz="0 1 0" />
+      <limit upper="1.7" lower="-1.7" effort="160" velocity="30" />
+    </joint>
+    <link name="link4">
+      <xacro:default_inertial/>
+      <visual>
+        <geometry>
+          <mesh filename="package://robotino_description/meshes/arm/link4.stl"/>
+        </geometry>
+        <material name="white" />
+        <origin rpy="0 0 0" xyz="0 0 0"/>
+      </visual>
+      <collision>
+        <origin rpy="0 0 0" xyz="0 0 0"/>
+        <geometry>
+          <mesh filename="package://robotino_description/meshes/arm/link4_collision.stl"/>
+        </geometry>
+      </collision>
+    </link>
+    <gazebo reference="link4">
+      <material>Gazebo/White</material>
+    </gazebo>
+    <joint name="joint5" type="revolute">
+      <parent link="link4"/>
+      <child link="link5"/>
+      <origin xyz="0.0 -0.027 0.035" rpy="0 0 0" />
+      <axis xyz="0 0 1" />
+      <limit upper="1.7" lower="-1.7" effort="160" velocity="30" />
+    </joint>
+    <link name="link5">
+      <xacro:default_inertial/>
+    </link>
+    <gazebo reference="link5">
+      <material>Gazebo/White</material>
+    </gazebo>
+  <xacro:arm_SimpleTransmission number="1"></xacro:arm_SimpleTransmission>
+  <xacro:arm_SimpleTransmission number="2"></xacro:arm_SimpleTransmission>
+  <xacro:arm_SimpleTransmission number="3"></xacro:arm_SimpleTransmission>
+  <xacro:arm_SimpleTransmission number="4"></xacro:arm_SimpleTransmission>
+  <xacro:arm_SimpleTransmission number="5"></xacro:arm_SimpleTransmission>
+  <xacro:arm_SimpleTransmission number="6"></xacro:arm_SimpleTransmission>
+  <xacro:arm_SimpleTransmission number="7"></xacro:arm_SimpleTransmission>
   </xacro:macro>
   <xacro:macro name="arm_SimpleTransmission" params="number">
     <transmission name="arm_${number}_trans">
       <type>transmission_interface/SimpleTransmission</type>
-      <joint name="arm_${number}_joint">
+      <joint name="joint${number}">
         <hardwareInterface>PositionJointInterface</hardwareInterface>
         <hardwareInterface>VelocityJointInterface</hardwareInterface>
@@ -20,209 +191,10 @@
     </transmission>
   </xacro:macro>
-  <xacro:macro name="arm" params="parent *origin">
-    <joint name="arm_base_joint" type="fixed">
-      <insert_block name="origin" />
-      <child link="arm_base_link" />
-      <parent link="${parent}"/>
-    </joint>
-    <link name="arm_base_link" >
-      <xacro:default_inertial/>
-      <visual>
-        <origin xyz="0.0 0.0 0.175" rpy="0 0.0 0.0" />
-        <geometry>
-          <cylinder radius="0.0" length="0.0"/>
-        </geometry>
-        <material name="LightGrey">
-          <color rgba="0.7 0.7 0.7 1.0"/>
-        </material>
-      </visual>
-      <collision>
-        <origin xyz="0.0 0.0 0.175" rpy="0 0.0 0.0" />
-        <geometry>
-          <cylinder radius="0.0" length="0.0"/>
-        </geometry>
-      </collision>
-    </link>
-    <joint name="arm_1_joint" type="revolute">
-      <parent link="arm_base_link" />
-      <child link = "arm_1_link" />
-      <origin xyz="0.0 0.0 0.0" rpy="0.0 0.0 0.0" />
-      <axis xyz="0 0 1" />
-      <calibration rising="${arm_1_ref}"/>
-      <limit effort="100" lower="-6.2831" upper="6.2831" velocity="1.4"/>
-    </joint>
-    <link name="arm_1_link">
-      <xacro:default_inertial/>
-      <visual>
-        <origin xyz="0.0 0.0 -0.04" rpy="0.0 0.0 0.0" />
-        <geometry>
-          <box size="0.08 0.08 0.08"/>
-        </geometry>
-        <material name="Black">
-          <color rgba="0 0 0 1.0"/>
-        </material>
-      </visual>
-      <collision>
-        <origin xyz="0.0 0.0 -0.04" rpy="0.0 0.0 0.0" />
-        <geometry>
-          <cylinder radius="0.025" length="0.08"/>
-        </geometry>
-      </collision>
-    </link>
-    <gazebo reference="arm_1_link">
-        <material>Gazebo/Black</material>
-    </gazebo>
-    <joint name="arm_2_joint" type="revolute">
-      <parent link="arm_1_link" />
-      <child link = "arm_2_link" />
-      <origin xyz="0.0 0.0 0.0" rpy="1.57 0.0 0.0" />
-      <axis xyz="0 0 1" />
-      <calibration rising="${arm_2_ref}"/>
-      <limit effort="100" lower="-2.36" upper="0.79" velocity="1.4"/>
-    </joint>
-    <link name="arm_2_link">
-      <xacro:default_inertial/>
-      <visual>
-        <origin xyz="0.0 0.125 0.0" rpy="1.57 0.0 0.0" />
-        <geometry>
-          <cylinder radius="0.025" length="0.25"/>
-        </geometry>
-        <material name="LightGrey">
-          <color rgba="0.7 0.7 0.7 1.0"/>
-        </material>
-      </visual>
-      <collision>
-        <origin xyz="0.0 0.125 0.0" rpy="1.57 0.0 0.0" />
-        <geometry>
-          <cylinder radius="0.025" length="0.25"/>
-        </geometry>
-      </collision>
-    </link>
-    <gazebo reference="arm_2_link">
-        <material>Gazebo/Grey</material>
-    </gazebo>
-    <joint name="arm_3_joint" type="revolute">
-      <parent link="arm_2_link" />
-      <child link = "arm_3_link" />
-      <origin xyz="0.0 0.25 -0.05" rpy="0.0 0.0 0.0" />
-      <axis xyz="0 0 1" />
-      <calibration rising="${arm_3_ref}"/>
-      <limit effort="100" lower="-2.62" upper="2.62" velocity="1.4"/>
-    </joint>
-    <link name="arm_3_link">
-      <xacro:default_inertial/>
-      <visual>
-        <origin xyz="0.0 0.125 0.0" rpy="-1.57 0.0 0.0" />
-        <geometry>
-          <cylinder radius="0.025" length="0.25"/>
-        </geometry>
-        <material name="Black">
-          <color rgba="0 0 0 1.0"/>
-        </material>
-      </visual>
-      <collision>
-        <origin xyz="0.0 0.125 0.0" rpy="-1.57 0.0 0.0" />
-        <geometry>
-          <cylinder radius="0.025" length="0.25"/>
-        </geometry>
-      </collision>
-    </link>
-    <gazebo reference="arm_3_link">
-        <material>Gazebo/Black</material>
-    </gazebo>
-    <joint name="arm_4_joint" type="revolute">
-      <parent link="arm_3_link" />
-      <child link = "arm_4_link" />
-      <origin xyz="0.0 0.175 0.0" rpy="-1.57 0.0 0.0" />
-      <axis xyz="0 0 1" />
-      <calibration rising="${arm_4_ref}"/>
-      <limit effort="100" lower="-2.62" upper="2.62" velocity="1.4"/>
-    </joint>
-    <link name="arm_4_link">
-      <xacro:default_inertial/>
-      <visual>
-        <origin xyz="0.0 0.0 -0.0375" rpy="0.0 0.0 0.0" />
-        <geometry>
-          <cylinder radius="0.04" length="0.05"/>
-        </geometry>
-        <material name="LightGrey">
-          <color rgba="0.7 0.7 0.7 1.0"/>
-        </material>
-      </visual>
-      <collision>
-        <origin xyz="0.0 0.0 -0.0375" rpy="0.0 0.0 0.0" />
-        <geometry>
-          <cylinder radius="0.04" length="0.05"/>
-        </geometry>
-      </collision>
-    </link>
-    <gazebo reference="arm_4_link">
-        <material>Gazebo/Grey</material>
-    </gazebo>
-    <joint name="arm_5_joint" type="revolute">
-      <parent link="arm_4_link" />
-      <child link = "arm_5_link" />
-      <origin xyz="0.0 0.05 0.075" rpy="1.57 0.0 0.0" />
-      <axis xyz="0 0 1" />
-      <calibration rising="${arm_5_ref}"/>
-      <limit effort="100" lower="-2.62" upper="2.62" velocity="1.4"/>
-    </joint>
-    <link name="arm_5_link">
-      <xacro:default_inertial/>
-      <visual>
-        <origin xyz="0.0 0.0175 0.0" rpy="-1.57 0.0 0.0" />
-        <geometry>
-          <cylinder radius="0.025" length="0.035"/>
-        </geometry>
-        <material name="Black">
-          <color rgba="0 0 0 1.0"/>
-        </material>
-      </visual>
-      <collision>
-        <origin xyz="0.0 0.0175 0.0" rpy="-1.57 0.0 0.0" />
-        <geometry>
-          <cylinder radius="0.025" length="0.035"/>
-        </geometry>
-      </collision>
-    </link>
-    <gazebo reference="arm_5_link">
-        <material>Gazebo/Black</material>
-    </gazebo>
-    <joint name="arm_6_joint" type="revolute">
-      <parent link="arm_5_link" />
-      <child link = "arm_6_link" />
-      <origin xyz="0.0 0.035 0.0" rpy="-1.57 0.0 0.0" />
-      <axis xyz="0 0 1" />
-      <calibration rising="${arm_6_ref}"/>
-      <limit effort="100" lower="-4.19" upper="4.19" velocity="1.4"/>
-    </joint>
-    <link name="arm_6_link">
-      <xacro:default_inertial/>
-      <visual>
-        <origin xyz="0.0 0.0 0.0125" rpy="0.0 0.0 0.0" />
-        <geometry>
-          <cylinder radius="0.025" length="0.025"/>
-        </geometry>
-        <material name="LightGrey">
-          <color rgba="0.7 0.7 0.7 1.0"/>
-        </material>
-      </visual>
-      <collision>
-        <origin xyz="0.0 0.0 -0.0125" rpy="0.0 0.0 0.0" />
-        <geometry>
-          <cylinder radius="0.025" length="0.025"/>
-        </geometry>
-      </collision>
-    </link>
-    <gazebo reference="arm_6_link">
-        <material>Gazebo/Grey</material>
-    </gazebo>
-    <xacro:arm_SimpleTransmission number="1"></xacro:arm_SimpleTransmission>
-    <xacro:arm_SimpleTransmission number="2"></xacro:arm_SimpleTransmission>
-    <xacro:arm_SimpleTransmission number="3"></xacro:arm_SimpleTransmission>
-    <xacro:arm_SimpleTransmission number="4"></xacro:arm_SimpleTransmission>
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
Commit message: update urdf

File: robotino_description/urdf/arm.urdf.xacro (robot description, xacro)
@@ -14,5 +14,5 @@
       </visual>
     </link>
-    <joint name="fixed_base_motor1" type="fixed">
+    <joint name="baserot" type="revolute">
       <parent link="base"/>
       <child link="motor1"/>

Commit message: fixed joint limits (pos and velocity)

File: robotino_description/urdf/arm.urdf.xacro (robot description, xacro)
@@ -31,5 +31,5 @@
       <origin xyz="0.0 0.0 0.0" rpy="0 0 0" />
       <axis xyz="0 1 0" />
-      <limit upper="1.5" lower="-1.2" effort="190" velocity="30" />
+      <limit upper="1.5" lower="-1.2" effort="190" velocity="0.7" />
     </joint>
     <link name="${name}link1">
@@ -57,5 +57,5 @@
       <origin xyz="0.0 0.0 0.25" rpy="0 0 0" />
       <axis xyz="0 1 0" />
-      <limit upper="2.3" lower="-1.7" effort="190" velocity="30" />
+      <limit upper="2.6" lower="-1.7" effort="190" velocity="0.7" />
     </joint>
     <link name="${name}motor2">
@@ -98,5 +98,5 @@
       <origin xyz="0.0 0.0 0.158" rpy="0 0 0" />
       <axis xyz="0 0 1" />
-      <limit upper="1.8" lower="-1.8" effort="190" velocity="30" />
+      <limit upper="1.8" lower="-1.8" effort="190" velocity="0.7" />
     </joint>
     <link name="${name}link3">
@@ -123,6 +123,6 @@
       <child link="${name}link4"/>
       <origin xyz="0.0 -0.057 0.065" rpy="0 0 0" />
-      <axis xyz="0 1 0" />
-      <limit upper="1.9" lower="-1.9" effort="160" velocity="30" />
+      <axis xyz="0 -1 0" />
+      <limit upper="2.4" lower="-2.4" effort="160" velocity="0.7" />
     </joint>
     <link name="${name}link4">
@@ -150,5 +150,5 @@
       <origin xyz="0.0 -0.027 0.035" rpy="0 0 0" />
       <axis xyz="0 0 1" />
-      <limit upper="2.9" lower="-2.9" effort="160" velocity="30" />
+      <limit upper="2.9" lower="-2.9" effort="160" velocity="0.7" />
     </joint>
     <link name="${name}link5">

Commit message: fix joint orientation

File: robotino_description/urdf/arm.urdf.xacro (robot description, xacro)
@@ -30,5 +30,5 @@
       <child link="${name}link1"/>
       <origin xyz="0.0 0.0 0.0" rpy="0 0 0" />
-      <axis xyz="0 1 0" />
+      <axis xyz="0 -1 0" />
       <limit upper="1.5" lower="-1.2" effort="190" velocity="0.7" />
     </joint>
