Commit message: updated the position of the collision  of the door

File: robotino_description/urdf/shell.urdf.xacro (robot description, xacro)
@@ -178,5 +178,5 @@
       </visual>
       <collision>
-        <origin xyz="0 0 0" rpy="0 0 0"/>
+        <origin xyz="-0.04 -0.01 0" rpy="0 0 0"/>
         <geometry>
           <mesh filename="package://robotino_description/meshes/door_collision.stl"/>
